File: SMPS hat production V1/SMPS hat/SMPS hat.sch (KiCad schematic (older format))
At the start: 22 parts, among them J2 Vin, J3 40HAT, J4 GPIO, J5 DISP, J6 DotStar, M1 Fan, Q4 Si4435, Q5 BSS138, U4 DS18S20Z, U5 74LVC125

Commit message: sync
Parts:
- removed J2: Vin, Connector_Phoenix_MSTB:PhoenixContact_MSTB_2,5_2-GF-5,08_1x02_P5.08mm_Horizontal_ThreadedFlange_MountHole, symbol Connector:Screw_Terminal_01x02
Connections:
- net +5V: now also J5.2 (Pin_2); no longer J5.3 (Pin_3)
- net GND: now also J5.1 (Pin_1); no longer J5.4 (Pin_4)
- net SCL: now also J5.4 (Pin_4); no longer J5.1 (Pin_1)
- net SDA: now also J5.3 (Pin_3); no longer J5.2 (Pin_2)
Changed lines of the file:
@@
 L Connector:Conn_01x04_Male J5
 U 1 1 5D4F978B
-P 4550 7000
-F 0 "J5" H 4658 7281 50  0000 C CNN
-F 1 "DISP" H 4658 7190 50  0000 C CNN
-F 2 "TerminalBlock_Phoenix:TerminalBlock_Phoenix_PT-1,5-4-3.5-H_1x04_P3.50mm_Horizontal" H 4550 7000 50  0001 C CNN
-F 3 "~" H 4550 7000 50  0001 C CNN
-	1    4550 7000
-	1    0    0    -1
+P 4550 7100
+F 0 "J5" H 4658 7381 50  0000 C CNN
+F 1 "DISP" H 4658 7290 50  0000 C CNN
+F 2 "TerminalBlock_Phoenix:TerminalBlock_Phoenix_PT-1,5-4-3.5-H_1x04_P3.50mm_Horizontal" H 4550 7100 50  0001 C CNN
+F 3 "~" H 4550 7100 50  0001 C CNN
+	1    4550 7100
+	1    0    0    1
 $EndComp
 Wire Wire Line
@@
 	1    0    0    -1
 $EndComp
-$Comp
-L Connector:Screw_Terminal_01x02 J2
-U 1 1 5D53F89A
-P 10250 4700
-F 0 "J2" H 10168 4375 50  0000 C CNN
-F 1 "Vin" H 10168 4466 50  0000 C CNN
-F 2 "Connector_Phoenix_MSTB:PhoenixContact_MSTB_2,5_2-GF-5,08_1x02_P5.08mm_Horizontal_ThreadedFlange_MountHole" H 10250 4700 50  0001 C CNN
-F 3 "~" H 10250 4700 50  0001 C CNN
-	1    10250 4700
-	-1   0    0    1
-$EndComp
-$Comp
-L power:GND #PWR0148
-U 1 1 5D540EF8
-P 10450 4700
-F 0 "#PWR0148" H 10450 4450 50  0001 C CNN
-F 1 "GND" H 10455 4527 50  0000 C CNN
-F 2 "" H 10450 4700 50  0001 C CNN
-F 3 "" H 10450 4700 50  0001 C CNN
-	1    10450 4700
-	1    0    0    -1
-$EndComp
 Text Label 6000 4400 2    50   ~ 0
 LED_SCLK
@@
 Text Label 2250 2700 1    50   ~ 0
 SCL
-Wire Wire Line
-	10450 4600 11600 4600
 $Comp
 L Device:R R6
@@
 	0    -1   -1   0
 $EndComp
-Text Label 11050 4600 0    50   ~ 0
-VIN
 $EndSCHEMATC
